File: AGB_LIPO.kicad_pcb (KiCad board)
At the start: 2 copper layers, 50 x 23 mm, 5 parts, among them J1 Conn_01x02_Male, U1 tp4056_board-tp4056

Commit message: Load Sharing and Voltage stabilizer
Parts:
- removed REF**: makho_fmask, misc_footprints:makho_fmask
- added  : AMS1117-3.3, Package_TO_SOT_SMD:SOT-223-3_TabPin2, F.Cu at (81.2, 28.8)
- added  : 100K, Resistor_THT:R_Axial_DIN0309_L9.0mm_D3.2mm_P15.24mm_Horizontal, F.Cu at (79.8, 22.3)
- added Q1: Si2319CDS, Package_TO_SOT_SMD:SOT-23, F.Cu at (92.4, 34.8)
- added TP1: TestPoint, TestPoint:TestPoint_THTPad_D1.0mm_Drill0.5mm, F.Cu at (89.6, 35.7)
- D1: footprint misc_footprints:Diode-hybrid-3pad -> Diode_THT:D_DO-34_SOD68_P7.62mm_Horizontal
- U1: value tp4056_board-tp4056 -> misc_tp4056_board-tp4056; footprint misc_footprints:4056E_LiIon_loader -> kiCad_mod:TP4056-18650
- moved D1 22.6 mm to (87.3, 34.3), turned to 180 degrees
- moved U1 16.7 mm to (96.5, 50.8)
Connections:
- J1 pad 2: Net-(D1-Pad1) -> Net-(J1-Pad2)
- U1 pad 5: Net-(D1-Pad2) -> Net-(Q1-Pad3)
Routing:
- net Net-(J1-Pad2): track 0.00 -> 53.1 mm, vias 0 -> 4
- net Net-(J1-Pad1): track 15.4 -> 55.8 mm
- net Net-(D1-Pad2): track 12.1 -> 24.7 mm
- net Net-(Q1-Pad3): track 0.00 -> 12.0 mm, vias 0 -> 1
- net Net-(D1-Pad1): track 22.8 -> 16.3 mm, vias 3 -> 1
Other:
- board text removed: "AGB_LIPO_ADAPTER https://github.com/makhowastaken/AGB_LIPO"
- board text removed: "This side down"

Commit message: Board updated
Parts:
- R1: renamed from  ; footprint Resistor_THT:R_Axial_DIN0309_L9.0mm_D3.2mm_P15.24mm_Horizontal -> Resistor_THT:R_Axial_DIN0204_L3.6mm_D1.6mm_P7.62mm_Horizontal
- U2: renamed from  
- moved TP1 1.45 mm to (89.4, 34.3)
Routing:
- net Net-(J1-Pad1): track 55.8 -> 63.4 mm
- net Net-(D1-Pad2): track 24.7 -> 26.4 mm
Other:
- board size 50 x 23 mm -> 49 x 23 mm
- board text added: "D1"
- board text added: "Q1"
- board text added: "R1"
- board text added: "THIS SIDE DOWN"

Commit message: 29/04 Update
Parts:
- added C1: 22u, Capacitor_Tantalum_SMD:CP_EIA-3216-18_Kemet-A, F.Cu at (116.3, 37.3)
- added C2: C, Capacitor_Tantalum_SMD:CP_EIA-3216-18_Kemet-A, F.Cu at (91.8, 27.4)
- added R2: 100, Resistor_THT:R_Axial_DIN0204_L3.6mm_D1.6mm_P7.62mm_Horizontal, F.Cu at (83.8, 36.6)
- moved TP1 9.23 mm to (95.4, 41.3)
- moved Q1 1.88 mm to (94.3, 34.9)
- moved R1 1.57 mm to (81.1, 23.2)
- moved D1 1.23 mm to (86.1, 34.3)
Connections:
- Q1 pad 1: Net-(D1-Pad2) -> Net-(Q1-Pad1)
Routing:
- net Net-(C1-Pad1): track 53.1 -> 67.6 mm, vias 4 -> 5
- net Net-(C2-Pad1): track 16.3 -> 27.9 mm, vias 1 -> 2
- net Net-(D1-Pad2): track 26.4 -> 34.1 mm, vias 0 -> 1
- net Net-(BT1-Pad1): track 31.8 -> 35.3 mm
- net Net-(Q1-Pad1): track 0.00 -> 2.29 mm
- net Net-(Q1-Pad3): track 12.0 -> 10.0 mm
- net Net-(C1-Pad2): track 63.4 -> 62.8 mm
Other:
- board text added: "+ -"
- board text added: "R2"
- board text removed: "B+ B-"
