File: AGB_LIPO.kicad_pcb (KiCad board)
At the start: 2 copper layers, 49 x 23 mm, 11 parts, among them J1 Conn_01x02_Male, Q1 Si2319CDS, U1 misc_tp4056_board-tp4056, U2 AMS1117-3.3

Commit message: 29/04 Symbol fix
Parts:
- C2: value C -> 10u
- Q1: value Si2319CDS -> Si2301DS
- moved C1 0.32 mm to (116.3, 37.7)
- moved C2 0.09 mm to (91.8, 27.4)
Changed lines of the file:
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@@
   )
   (module Capacitor_Tantalum_SMD:CP_EIA-3216-18_Kemet-A (layer F.Cu)
-    (at 91.7575 27.432 180)
+    (at 91.821 27.3685 180)
     (descr "Tantalum Capacitor SMD Kemet-A (3216-18 Metric), IPC_7351 nominal, (Body size from: http://www.kemet.com/Lists/ProductCatalog/Attachments/253/KEM_TC101_STD.pdf), generated with kicad-footprint-generator")
     (tags "capacitor tantalum")
     (attr smd)
-    (fp_text reference C2 (at 0.0635 -0.127) (layer F.SilkS)
-      (effects (font (size 1 1) (thickness 0.15)))
-    )
-    (fp_text value C (at 0 1.75) (layer F.Fab)
+    (fp_text reference C2 (at -0.127 0) (layer F.SilkS)
+      (effects (font (size 1 1) (thickness 0.15)))
+    )
+    (fp_text value 10u (at 0 1.75) (layer F.Fab)
       (effects (font (size 1 1) (thickness 0.15)))
     )
@@
   )
   (module Capacitor_Tantalum_SMD:CP_EIA-3216-18_Kemet-A (layer F.Cu)
-    (at 116.2685 37.338 90)
+    (at 116.2685 37.6555 90)
     (descr "Tantalum Capacitor SMD Kemet-A (3216-18 Metric), IPC_7351 nominal, (Body size from: http://www.kemet.com/Lists/ProductCatalog/Attachments/253/KEM_TC101_STD.pdf), generated with kicad-footprint-generator")
     (tags "capacitor tantalum")
     (attr smd)
-    (fp_text reference C1 (at 0 -0.127 90) (layer F.SilkS)
+    (fp_text reference C1 (at 0 -0.0635 90) (layer F.SilkS)
       (effects (font (size 1 1) (thickness 0.15)))
     )
@@
       (effects (font (size 1 1) (thickness 0.15)))
     )
-    (fp_text value Si2319CDS (at 0 2.5 90) (layer F.Fab)
-      (effects (font (size 1 1) (thickness 0.15)))
-    )
+    (fp_text value Si2301DS (at 0 2.5 90) (layer F.Fab)
+      (effects (font (size 1 1) (thickness 0.15)))
+    )

Commit message: Full Circuit redesign
Parts:
- added C3: 220u, Capacitor_Tantalum_SMD:CP_EIA-3528-21_Kemet-B, F.Cu at (91.5, 24.8)
- C1: value 22u -> 4,7u; footprint Capacitor_Tantalum_SMD:CP_EIA-3216-18_Kemet-A -> Capacitor_SMD:C_0603_1608Metric
- C2: value 10u -> 4,7u; footprint Capacitor_Tantalum_SMD:CP_EIA-3216-18_Kemet-A -> Capacitor_SMD:C_0603_1608Metric
- U2: value AMS1117-3.3 -> AP2114H-3_3TRG1; footprint Package_TO_SOT_SMD:SOT-223-3_TabPin2 -> digikey-footprints:SOT-223
- moved C1 37.4 mm to (79.1, 33.5), turned to 180 degrees
- moved C2 12.9 mm to (79.9, 22.4)
- moved R1 10.7 mm to (91.6, 21.1), turned to 180 degrees
- moved D1 5.88 mm to (91.4, 36.9)
- moved R2 1.91 mm to (83.8, 34.7)
- moved U2 1.18 mm to (80.6, 27.7), turned to 0 degrees
- moved Q1 0.64 mm to (94.4, 35.5), turned to 0 degrees
Connections:
- D1 pad 1: Net-(C2-Pad1) -> Net-(C1-Pad1)
- J1 pad 2: Net-(C1-Pad1) -> Net-(C2-Pad1)
- Q1 pad 2: Net-(C2-Pad1) -> Net-(C1-Pad1)
- U2 pad 2: Net-(C1-Pad1) -> (no net)
- U2 pad 3: Net-(C2-Pad1) -> Net-(C1-Pad1)
Routing:
- net Net-(C1-Pad1): track 67.6 -> 17.6 mm, vias 5 -> 0
- net Net-(C2-Pad1): track 27.9 -> 51.1 mm, vias 2 -> 3
- net Net-(C1-Pad2): track 62.8 -> 71.9 mm, vias 1 -> 2
- net Net-(D1-Pad2): track 34.1 -> 33.4 mm, vias 1 -> 2
- net Net-(Q1-Pad3): track 10.0 -> 10.5 mm, vias 1 -> 0
- added copper zone on F.Cu, net Net-(C1-Pad2)

Commit message: 17.06 UPDATE
Parts:
- removed Q1: Si2301DS, Package_TO_SOT_SMD:SOT-23
- added C4: 220u, Capacitor_Tantalum_SMD:CP_EIA-3528-21_Kemet-B_Pad1.50x2.35mm_HandSolder, F.Cu at (118.5, 94.9)
- added D2: 1N4001, SamacSys_Parts:DIOM5626X245N, F.Cu at (133.5, 110.4)
- added IC1: LP38693MP-ADJ_NOPB, SamacSys_Parts:SOT150P700X180-5N, F.Cu at (128.8, 101.2)
- added R3: 1M, Resistor_SMD:R_0603_1608Metric_Pad1.05x0.95mm_HandSolder, F.Cu at (122.6, 100.3)
- added R4: 270k, Resistor_SMD:R_0805_2012Metric_Pad1.15x1.40mm_HandSolder, F.Cu at (127.2, 108.8)
- added R5: 240k, Resistor_SMD:R_0805_2012Metric_Pad1.15x1.40mm_HandSolder, F.Cu at (128.0, 111.1)
- C1: value 4,7u -> 4u7; footprint Capacitor_SMD:C_0603_1608Metric -> Capacitor_SMD:C_0603_1608Metric_Pad1.05x0.95mm_HandSolder
- C2: value 4,7u -> 10u; footprint Capacitor_SMD:C_0603_1608Metric -> Capacitor_SMD:C_0603_1608Metric_Pad1.05x0.95mm_HandSolder
- C3: value 220u -> 4u7; footprint Capacitor_Tantalum_SMD:CP_EIA-3528-21_Kemet-B -> Capacitor_SMD:C_0603_1608Metric_Pad1.05x0.95mm_HandSolder
- D1: value D -> 1N4001; footprint Diode_THT:D_DO-34_SOD68_P7.62mm_Horizontal -> SamacSys_Parts:DIOM5626X245N
- R1: value 100K -> 470k; footprint Resistor_THT:R_Axial_DIN0204_L3.6mm_D1.6mm_P7.62mm_Horizontal -> Resistor_SMD:R_0603_1608Metric_Pad1.05x0.95mm_HandSolder
- R2: value 100 -> 62k; footprint Resistor_THT:R_Axial_DIN0204_L3.6mm_D1.6mm_P7.62mm_Horizontal -> Resistor_SMD:R_0805_2012Metric_Pad1.15x1.40mm_HandSolder
- TP1: footprint TestPoint:TestPoint_THTPad_D1.0mm_Drill0.5mm -> TestPoint:TestPoint_Loop_D1.80mm_Drill1.0mm_Beaded
- U1: value misc_tp4056_board-tp4056 -> tp4056_board-tp4056; footprint kiCad_mod:TP4056-18650 -> digikey-footprints:4056E_LiIon_loader; moved to B.Cu
- U2: value AP2114H-3_3TRG1 -> TPS3700DDCR; footprint digikey-footprints:SOT-223 -> SamacSys_Parts:SOT98P280X110-6N
- moved R1 98.5 mm to (126.0, 113.4)
- moved R2 86.5 mm to (123.2, 111.7)
- moved C2 85.4 mm to (120.4, 97.5)
- moved C3 84.8 mm to (133.6, 98.4), turned to 90 degrees
- moved C1 84.2 mm to (124.2, 104.6), turned to 270 degrees
- moved J1 82.1 mm to (155.6, 104.1)
- moved BT1 81.6 mm to (115.8, 109.8)
- moved U2 81.0 mm to (116.8, 100.1), turned to 270 degrees
- moved U1 73.2 mm to (145.2, 105.4)
- moved D1 67.4 mm to (127.7, 93.6), turned to 0 degrees
- moved TP1 64.4 mm to (133.3, 93.4)
Connections:
- C1 pad 2: Net-(C1-Pad2) -> GND
- C2 pad 2: Net-(C1-Pad2) -> GND
- C3 pad 1: Net-(C2-Pad1) -> GND
- C3 pad 2: Net-(C1-Pad2) -> Net-(C3-Pad2)
- J1 pad 1: Net-(C1-Pad2) -> GND
- J1 pad 2: Net-(C2-Pad1) -> Net-(C3-Pad2)
- R1 pad 1: Net-(D1-Pad2) -> Net-(D2-Pad2)
- R1 pad 2: Net-(C1-Pad2) -> Net-(R1-Pad2)
- R2 pad 1: Net-(D1-Pad2) -> Net-(R1-Pad2)
- R2 pad 2: Net-(Q1-Pad1) -> GND
- U1 pad 5: Net-(Q1-Pad3) -> Net-(D2-Pad2)
- U1 pad 6: Net-(C1-Pad2) -> GND
- U2 pad 1: Net-(C1-Pad2) -> (no net)
- U2 pad 2: (no net) -> GND
- U2 pad 3: Net-(C1-Pad1) -> GND
- U2 pad 4: Net-(C2-Pad1) -> Net-(R1-Pad2)
Routing:
- net GND: track 0.00 -> 114.6 mm, vias 0 -> 6
- net Net-(C3-Pad2): track 0.00 -> 76.4 mm, vias 0 -> 6
- net Net-(C1-Pad2): track 71.9 -> 0.00 mm, vias 2 -> 0
- net Net-(D2-Pad2): track 0.00 -> 48.1 mm, vias 0 -> 1
- net Net-(C1-Pad1): track 17.6 -> 61.8 mm, vias 0 -> 5
- net Net-(C2-Pad1): track 51.1 -> 7.99 mm, vias 3 -> 0
- net Net-(IC1-Pad2): track 0.00 -> 30.7 mm, vias 0 -> 2
- net Net-(D1-Pad2): track 33.4 -> 3.70 mm, vias 2 -> 0
- net Net-(R1-Pad2): track 0.00 -> 18.2 mm
- net Net-(BT1-Pad1): track 35.3 -> 48.0 mm, vias 0 -> 2
- net Net-(Q1-Pad3): track 10.5 -> 0.00 mm
- net Net-(BT1-Pad2): track 37.9 -> 43.9 mm, vias 0 -> 1
- net Net-(J1-Pad1): track 0.00 -> 5.05 mm, vias 0 -> 5
- net Net-(D1-Pad1): track 0.00 -> 5.05 mm, vias 0 -> 5
- net Net-(Q1-Pad1): track 2.06 -> 0.00 mm
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- added copper zone on B.Cu, net GND
- added copper zone on F.Cu, net GND
- removed copper zone on F.Cu, net Net-(C1-Pad2)
Other:
- board size 49 x 23 mm -> 50 x 25.3 mm
- board text added: "B+ B-"
- board text added: "Based on Makho's board. https://github.com/makhowastaken/AGB_LIPO Recreated by Lobod. https://github.com/LobodPl/AGB_LIPO"
- board text added: "This side down do not eat"
- board text removed: "+ -"
- board text removed: "D1"
- board text removed: "Q1"
- board text removed: "R1"
- board text removed: "R2"
- board text removed: "THIS SIDE DOWN"
